File: buzzerpi/board_ätzen.brd (EAGLE design)
At the start: 100 x 80 mm, 11 parts, among them IC1 ULN2003AN, IC2 ULN2003AN

Commit message: geändert
Parts:
- X3: device con-ptr500:AK500/8 -> con-ptr500:AK500/10
- moved U$5 96.9 mm to (63.5, 61.0), turned to 180 degrees
- moved U$4 77.2 mm to (63.5, 48.3), turned to 180 degrees
- moved U$1 43.3 mm to (63.5, 14.0)
- moved U$2 16.9 mm to (63.5, 25.4)
- moved IC1 11.4 mm to (43.2, 53.3)
- moved U$3 10.9 mm to (63.5, 36.8), turned to 180 degrees
- moved X3 3.59 mm to (91.4, 39.4)
Connections:
- removed net N$19 (its old number): IC1.13, U$1.COIL1
- removed net N$20 (its old number): IC1.10, U$3.COIL1
- removed net N$28 (its old number): U$1.CON1OPTION, X3.6
- new net N$21: IC1.13, U$3.COIL1
- new net N$26: U$4.CON1OPTION, X3.8
- new net N$30: IC1.10, U$1.COIL1
- new net N$31: U$2.CENTER1, X3.3
- new net N$32: U$1.CON1OPTION, X3.2
- new net N$33: U$1.CENTER1, X3.1
- new net N$34: U$5.CON1OPTION, X3.10
- net N$22: now also U$4.CENTER1, X3.7; no longer U$3.CENTER2, X3.1
- net N$23: now also X3.6; no longer X3.2
- net N$25: now also U$5.CENTER1, X3.9; no longer U$2.CENTER2, X3.3
- net N$27: now also U$3.CENTER1; no longer U$1.CENTER2
Routing:
- net N$30: track 0.00 -> 42.0 mm
- net N$32: track 0.00 -> 38.5 mm
- net N$28: track 0.00 -> 37.9 mm
- net N$23: track 0.00 -> 37.3 mm
- net N$26: track 0.00 -> 36.7 mm
- net N$34: track 0.00 -> 35.9 mm
- net N$24: track 0.00 -> 33.0 mm
- net GND: track 0.00 -> 27.2 mm
- net N$21: track 0.00 -> 26.7 mm
- net N$33: track 0.00 -> 24.8 mm
- net N$31: track 0.00 -> 24.2 mm
- net N$27: track 0.00 -> 23.6 mm
- net N$22: track 0.00 -> 23.0 mm
- net N$25: track 0.00 -> 22.1 mm
- net N$20: track 0.00 -> 17.7 mm
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- added copper zone on layer 16, net +5V
