File: buzzerpi/board_ätzen.sch (EAGLE design)
At the start: 11 parts, among them IC1 ULN2003AN, IC2 ULN2003AN

Commit message: geändert
Parts:
- X3: device con-ptr500:AK500/8 -> con-ptr500:AK500/10
Connections:
- removed net N$19 (its old number): IC1.O4, U$1G$1.1
- removed net N$20 (its old number): IC1.O7, U$3G$1.1
- removed net N$28 (its old number): U$1G$2.S, X3-6.KL
- new net N$21: IC1.O4, U$3G$1.1
- new net N$26: U$4G$2.S, X3-8.KL
- new net N$30: IC1.O7, U$1G$1.1
- new net N$31: U$2G$2.P@1, X3-3.KL
- new net N$32: U$1G$2.S, X3-2.KL
- new net N$33: U$1G$2.P@1, X3-1.KL
- new net N$34: U$5G$2.S, X3-10.KL
- net N$22: now also U$4G$2.P@1, X3-7.KL; no longer U$3G$2.P, X3-1.KL
- net N$23: now also X3-6.KL; no longer X3-2.KL
- net N$25: now also U$5G$2.P@1, X3-9.KL; no longer U$2G$2.P, X3-3.KL
- net N$27: now also U$3G$2.P@1; no longer U$1G$2.P
Other:
- moved on the sheet: U$1, U$2, U$3, U$4, U$5, X3-1, X3-2, X3-3, X3-4, X3-5, X3-6, X3-7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
